File: StartClock/StartClock.kicad_sch (KiCad schematic)
At the start: 49 parts, among them J1 Screw_Terminal_01x05, J2 Screw_Terminal_01x02, J3 Screw_Terminal_01x02, J4 Screw_Terminal_01x02, J5 Screw_Terminal_01x04, Q1 2STR1160, Q2 2STR1160, SW1 SW_Omron_B3FS, SW2 SW_Omron_B3FS, SW3 SW_Omron_B3FS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

Commit message: Components updates after Mouser ordering few parts changed due to unavailability
Parts:
- C8: value 50n -> 0.047u
- J1, J5: Ref mouser https://www.mouser.fr/ProductDetail/Phoenix-Contact/1725685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 -> https://www.mouser.fr/ProductDetail/Wurth-Elektronik/691210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
- J2, J3, J4: Ref mouser https://www.mouser.fr/ProductDetail/Phoenix-Contact/1725656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 -> https://www.mouser.fr/ProductDetail/Wurth-Elektronik/691210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
- R12: footprint Resistor_SMD:R_1210_3225Metric_Pad1.30x2.65mm_HandSolder -> Resistor_SMD:R_2512_6332Metric; Ref mouser https://www.mouser.fr/ProductDetail/YAGEO/AC1210FR-7W220RL?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 -> https://www.mouser.fr/ProductDetail/YAGEO/RC2512FK-07220RL?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
Changed lines of the file:
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@@
 			)
 		)
-		(property "Ref mouser" "https://www.mouser.fr/ProductDetail/Phoenix-Contact/1725656?qs=Ul7CXFMnlWWQeccayYbRmw%3D%3D"
+		(property "Ref mouser" "https://www.mouser.fr/ProductDetail/Wurth-Elektronik/691210910002?qs=sPbYRqrBIVlpmUgpxfjjUA%3D%3D"
 			(at 149.86 180.34 0)
 			(effects
@@
 			)
 		)
-		(property "Ref mouser" "https://www.mouser.fr/ProductDetail/Phoenix-Contact/1725656?qs=Ul7CXFMnlWWQeccayYbRmw%3D%3D"
+		(property "Ref mouser" "https://www.mouser.fr/ProductDetail/Wurth-Elektronik/691210910002?qs=sPbYRqrBIVlpmUgpxfjjUA%3D%3D"
 			(at 259.08 154.94 0)
 			(effects
@@
 			)
 		)
-		(property "Footprint" "Resistor_SMD:R_1210_3225Metric_Pad1.30x2.65mm_HandSolder"
+		(property "Footprint" "Resistor_SMD:R_2512_6332Metric"
 			(at 129.794 83.566 90)
 			(effects
@@
 			)
 		)
-		(property "Ref mouser" "https://www.mouser.fr/ProductDetail/YAGEO/AC1210FR-7W220RL?qs=r5DSvlrkXmJYQoM71ylR%2FQ%3D%3D"
+		(property "Ref mouser" "https://www.mouser.fr/ProductDetail/YAGEO/RC2512FK-07220RL?qs=GMd7ukQor4OMhGSsbk8aRQ%3D%3D"
 			(at 130.81 83.82 0)
 			(effects
@@
 			)
 		)
-		(property "Ref mouser" "https://www.mouser.fr/ProductDetail/Phoenix-Contact/1725656?qs=Ul7CXFMnlWWQeccayYbRmw%3D%3D"
+		(property "Ref mouser" "https://www.mouser.fr/ProductDetail/Wurth-Elektronik/691210910002?qs=sPbYRqrBIVlpmUgpxfjjUA%3D%3D"
 			(at 143.51 90.17 0)
 			(effects
@@
 			)
 		)
-		(property "Value" "50n"
+		(property "Value" "0.047u"
 			(at 242.57 138.4299 0)
 			(effects
@@
 			)
 		)
-		(property "Ref mouser" "https://www.mouser.fr/ProductDetail/Phoenix-Contact/1725685?qs=A%2FKWGUWTCZiuYWt6zAMYZA%3D%3D"
+		(property "Ref mouser" "https://www.mouser.fr/ProductDetail/Wurth-Elektronik/691210910005?qs=sPbYRqrBIVmsC84njkCQMg%3D%3D"
 			(at 237.49 81.28 0)
 			(effects
@@
 			)
 		)
-		(property "Ref mouser" "https://www.mouser.fr/ProductDetail/Phoenix-Contact/1725685?qs=A%2FKWGUWTCZiuYWt6zAMYZA%3D%3D"
+		(property "Ref mouser" "https://www.mouser.fr/ProductDetail/Wurth-Elektronik/691210910004?qs=sPbYRqrBIVlxffWXw70IkA%3D%3D"
 			(at 30.48 177.8 0)
 			(effects
